File: KC-ETAclock-5v/ETAclock.kicad_pcb (KiCad board)
At the start: 2 copper layers, 240 x 38.7 mm, 126 parts, among them J1 Conn_01x01, J2 Conn_01x01, J3 Conn_01x01, J4 Conn_01x01, J5 USB_SUPPLY, J6 Conn_01x05, P15 Raspberry_PI_Zero_Hat, Q10 MMBTA42, Q11 MMBT3906, Q12 MMBTA42, Q13 MMBT3906, Q14 MMBTA42, Q15 MMBT3906, Q16 MMBTA42, Q17 MMBT3906, Q18 MMBTA42, Q19 MMBT3906, Q2 MMBTA42, Q20 MMBTA42, Q21 MMBT3906, Q22 MMBTA42, Q23 MMBT3906, Q24 MMBTA42, Q25 MMBT3906, Q3 MMBT3906, Q4 MMBTA42, Q5 MMBT3906, Q6 MMBTA42, Q7 MMBT3906, Q8 MMBTA42, Q9 MMBT3906, U10 IN-4, U11 TPIC6B595, U12 IN-4, U13 IN-4, U14 TPIC6B595, U3 IN-4, U4 TPIC6B595, U5 IN-4, U6 74HCT04, U7 TPIC6B595, U8 IN-4, U9 TPIC6B595

Commit message: The TestDigits.py is a script file that allows for the following feastures:
- cycle through all digits 1 second at a time
- display any single digit
- burn in all digits
- burn in even digits
- burn in odd digits
- toggle N_DISABLE
- toggle POWER

here is the command from the python script.

 print("press:")
   print("return: to index the displayed diget to the next value")
   print("[t]: to start time 1-9:")
   print("[T]: For a x minute burn in of all digits")
   print("[0-9]: to display the digit to light up")
   print("[d]: to toggle display N_DISABLE")
   print("[p]: to toggle the power supply on/off")
   print("[OT]: for a x minute burn in of odd digits (for biquaniary driven tubes")
   print("[ET]: for a x minute burn in of even digits (for biquinary driven tubes)")
   print("[x]: to exit program")
Parts:
- moved ? 21.9 mm to (111.4, 105.4)
- moved ? 21.9 mm to (101.5, 101.1)
- moved C19 21.9 mm to (56.5, 89.3)
- moved C2 21.9 mm to (93.0, 80.6)
- moved C24 21.9 mm to (98.3, 94.9)
- moved C25 21.9 mm to (138.9, 94.4)
- moved C26 21.9 mm to (179.6, 94.0)
- moved C28 21.9 mm to (246.3, 104.2)
- moved C3 21.9 mm to (136.9, 78.7)
- moved C31 21.9 mm to (141.0, 94.3)
- moved C32 21.9 mm to (182.3, 94.0)
- moved C33 21.9 mm to (223.5, 87.6)
- moved C4 21.9 mm to (178.3, 79.1)
- moved C5 21.9 mm to (222.4, 77.7)
- moved J1 21.9 mm to (26.7, 109.9)
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